Commit message: Release/Flexiv ROS 2 Humble v1.5 (#40)

File: flexiv_description/urdf/rizon.urdf.xacro (robot description, xacro)
@@ -10,4 +10,5 @@
   <xacro:arg name="prefix" default="" />
   <xacro:arg name="robot_sn" default="" />
+  <xacro:arg name="load_gripper" default="false" />
   <xacro:arg name="use_fake_hardware" default="false" />
   <xacro:arg name="fake_sensor_commands" default="false" />
@@ -19,4 +20,5 @@
     prefix="$(arg prefix)"
     robot_sn="$(arg robot_sn)"
+    load_gripper="$(arg load_gripper)"
     use_fake_hardware="$(arg use_fake_hardware)"
     fake_sensor_commands="$(arg fake_sensor_commands)"

File: flexiv_description/urdf/rizon_macro.xacro (robot description, xacro)
@@ -5,8 +5,14 @@
     prefix
     robot_sn
+    load_gripper:=false
     use_fake_hardware:=false
     fake_sensor_commands:=false
     initial_positions:=${dict(joint1=0.0,joint2=-0.69813,joint3=0.0,joint4=1.570796,joint5=0.0,joint6=0.69813,joint7=0.0)}
     ">
+    <!-- Load gripper -->
+    <xacro:if value="${load_gripper}">
+      <xacro:include filename="$(find flexiv_description)/urdf/grav_macro.xacro" />
+      <xacro:flexiv_GN01 prefix="${prefix}" mesh_prefix_path="package://flexiv_description/" />
+    </xacro:if>
     <!-- Import Rviz colors -->
     <xacro:include filename="$(find flexiv_description)/urdf/flexiv_arm.materials.xacro" />

File: flexiv_moveit_config/srdf/rizon.srdf.xacro (robot description, xacro)
@@ -1,9 +1,16 @@
 <?xml version="1.0" encoding="UTF-8"?>
-<robot xmlns:xacro="http://wiki.ros.org/xacro" name="$(arg name)">
+<robot xmlns:xacro="http://wiki.ros.org/xacro" name="(arg name)">
     <!-- robot name parameter -->
-    <xacro:arg name="name" default="rizon"/>
+    <xacro:arg name="name" default="rizon" />
     <!-- parameters -->
     <xacro:arg name="prefix" default="" />
-    <xacro:include filename="$(find flexiv_moveit_config)/srdf/rizon_macro.srdf.xacro"/>
-    <xacro:rizon_srdf name="$(arg name)" prefix="$(arg prefix)"/>
+    <xacro:arg name="load_gripper" default="false" />
+    <xacro:property name="name" value="$(arg name)"/>
+    <xacro:include filename="$(find flexiv_moveit_config)/srdf/rizon_macro.srdf.xacro" />
+    <xacro:rizon_srdf name="${name}" prefix="$(arg prefix)" />
+    <!-- Load gripper -->
+    <xacro:if value="$(arg load_gripper)">
+        <xacro:include filename="$(find flexiv_moveit_config)/srdf/grav.srdf.xacro" />
+        <xacro:grav_srdf name="${name}" prefix="$(arg prefix)" />
+    </xacro:if>
 </robot>
